Commit message: intialize 0.475 0.1092 0.42

File: Robots/universalUR5/sm_universalUR5.urdf (robot description, URDF)
Before this commit: robot ur5, 11 links, 10 joints
Joints:
- joint elbow_joint: origin xyz=0.0 -0.1197 0.425 rpy=0.0 0.0 0.0 -> xyz=0.0 -0.1197 0.425 rpy=0.0 1.57079632679 0.0
- joint shoulder_lift_joint: origin xyz=0.0 0.13585 0.0 rpy=0.0 1.57079632679 0.0 -> xyz=0.0 0.13585 0.0 rpy=0.0 0.0 0.0
- joint wrist_2_joint: origin xyz=0.0 0.093 0.0 rpy=0.0 0.0 0.0 -> xyz=0.0 0.093 0.0 rpy=0.0 0.0 1.57079632679
